File: hardware/photo_frame.kicad_sch (KiCad schematic)
At the start: 27 parts, among them J1 Micro_SD_Card, J3 Conn_01x03_Pin, Q3 Q_PMOS_GSD, Q4 Q_PMOS_GSD, SW1 SW_Push, SW2 SW_Push, SW3 SW_Push, U1 STM32L010K8Tx, Y1 32.768k

Commit message: Refactored hardware - finished design v1
Parts:
- removed J1: Micro_SD_Card, symbol Connector:Micro_SD_Card
- added J1: Micro_SD_Card_Det2, photo_frame:TFP09-2-12B, symbol Connector:Micro_SD_Card_Det2
- added Q5: FDN306P, Package_TO_SOT_SMD:SOT-23-3, symbol Device:Q_PMOS_GSD
- BT1: footprint (none) -> photo_frame:BAT_BK-877
- C6, C7: value 10p -> 6p
- Q3, Q4: value Q_PMOS_GSD -> FDN306P; footprint (none) -> Package_TO_SOT_SMD:SOT-23-3
- SW1, SW2, SW3: footprint (none) -> Button_Switch_SMD:SW_SPST_EVQP2
- Y1: footprint (none) -> Crystal:Crystal_SMD_Abracon_ABS25-4Pin_8.0x3.8mm; symbol Device:Crystal_Small -> Device:Crystal_GND23_Small
Connections:
- net GND: now also J3.1 (Pin_1), J1.11 (SHIELD), J1.6 (VSS), Q5.1 (G); no longer J3.3 (Pin_3)
- net SPI_MISO: now also J1.7 (DAT0)
- net SPI_MOSI: now also J1.3 (CMD)
- net SPI_SCK: now also J1.5 (CLK)
- net SPI_SD_CS: now also U1.30 (PB7), J1.2 (DAT3/CD)
- net SWDIO: now also J3.3 (Pin_3); no longer J3.1 (Pin_1)
- net VDD: now also Q5.2 (S); no longer BT1.1 (+), R3.2, R4.2, R5.2, R6.2
- net at C7.1, U1.3 (PC15): now also Y1.4; no longer Y1.2
- net at R3.1: now also J1.1 (DAT2)
- net SD_VDD: now reaches Q4.3 (D)
- net SD_VDD: now also R3.2, R4.2, R5.2, R6.2, J1.4 (VDD)
- net at R6.1: now also J1.8 (DAT1)
- new net +BATT: BT1.1 (+), Q5.3 (D)
- no-connect marks 11 -> 14
Other:
- moved on the sheet: BT1, J3
